Commit message: teleop and simulation

File: description/robot.urdf.xacro (robot description, xacro)
@@ -2,3 +2,4 @@
 <robot xmlns:xacro="http://www.ros.org/wiki/xacro"  name="robot">
     <xacro:include filename="robot_core.xacro" />
+    <xacro:include filename="gazebo_control.xacro"/>
 </robot>

File: description/robot_core.xacro (robot description, xacro)
@@ -5,107 +5,112 @@
         <color rgba="1 1 1 1"/>
     </material>
-    <material name = "orange">
+    <material name="orange">
         <color rgba="1 0.3 0.1 1"/>
     </material>
-    <material name = "blue">
-        <color rgba = "0.2 0.2 1 1"/>
+    <material name="blue">
+        <color rgba="0.2 0.2 1 1"/>
     </material>
-    <material name = "black">
-        <color rgba = "0 0 0 1"/>
+    <material name="black">
+        <color rgba="0 0 0 1"/>
     </material>
-    <!-- BASE LINK -->
     <link name="base_link">
     </link>
-    <!-- CHASSIS LINK -->
-    <joint name = "chassis_joint" type = "fixed">
-        <parent link = "base_link"/>
-        <child link = "chassis"/>
-        <origin xyz = "-0.1 0 0"/>
+    <!-- CHASSIS -->
+    <joint name="chassis_joint" type="fixed">
+        <parent link="base_link"/>
+        <child link="chassis"/>
+        <origin xyz="-0.1 0 0"/>
     </joint>
-    <link name = "chassis">
+    <link name="chassis">
         <visual>
-            <origin xyz = "0.15 0 0.075"/>
+            <origin xyz="0.15 0 0.075" rpy="0 0 0"/>
             <geometry>
-                <box size = "0.3 0.3 0.15"/>
+                <box size="0.3 0.3 0.15"/>
             </geometry>
-            <material name = "white"/>
+            <material name="white"/>
         </visual>
         <collision>
-            <origin xyz = "0.15 0 0.075"/>
+            <origin xyz="0.15 0 0.075" rpy="0 0 0"/>
             <geometry>
-                <box size = "0.3 0.3 0.15"/>
+                <box size="0.3 0.3 0.15"/>
             </geometry>
         </collision>
-        <xacro:inertial_box mass = "1.0" x = "0.3" y = "0.3" z = "0.15">
-            <origin xyz = "0.15 0 0.075" rpy = "0 0 0"/>
+        <xacro:inertial_box mass="0.5" x="0.3" y="0.3" z="0.15">
+            <origin xyz="0.15 0 0.075" rpy="0 0 0"/>
         </xacro:inertial_box>
     </link>
-    <!-- LEFT WHEEL LINK -->
-    <joint name = "left_wheel_joint" type = "continuous">
-        <parent link = "base_link"/>
-        <child link = "left_wheel"/>
-        <origin xyz = "0 0.175 0" rpy = "-${pi/2} 0 0"/>
-        <axis xyz = "0 0 1"/>
+    <!-- LEFT WHEEL -->
+    <joint name="left_wheel_joint" type="continuous">
+        <parent link="base_link"/>
+        <child link="left_wheel"/>
+        <origin xyz="0 0.175 0" rpy="-${pi/2} 0 0"/>
+        <axis xyz="0 0 1"/>
+        <limit effort="0.05" velocity="10.0"/>
     </joint>
-    <link name = "left_wheel">
+    <link name="left_wheel">
         <visual>
             <geometry>
-                <cylinder radius = "0.05" length = "0.04"/>
+                <cylinder length="0.04" radius="0.05" />
             </geometry>
-            <material name = "blue"/>
+            <material name="blue"/>
         </visual>
         <collision>
             <geometry>
-                <cylinder radius = "0.05" length = "0.04"/>
+                <sphere radius="0.05" />
             </geometry>
         </collision>
-        <xacro:inertial_cylinder mass = "1.0" length = "0.04" radius = "0.05">
-            <origin xyz = "0 0 0" rpy = "0 0 0"/>
+        <xacro:inertial_cylinder mass="0.1" length="0.04" radius="0.05">
+            <origin xyz="0 0 0" rpy="0 0 0"/>
         </xacro:inertial_cylinder>
     </link>
-        <!-- RIGHT WHEEL LINK -->
-    <joint name = "right_wheel_joint" type = "continuous">
-        <parent link = "base_link"/>
-        <child link = "right_wheel"/>
-        <origin xyz = "0 -0.175 0" rpy = "${pi/2} 0 0"/>
-        <axis xyz = "0 0 -1"/>
+    <!-- RIGHT WHEEL -->
+    <joint name="right_wheel_joint" type="continuous">
+        <parent link="base_link"/>
+        <child link="right_wheel"/>
+        <origin xyz="0 -0.175 0" rpy="${pi/2} 0 0"/>
+        <axis xyz="0 0 -1"/>
+        <limit effort="0.05" velocity="10.0"/>
     </joint>
-    <link name = "right_wheel">
+    <link name="right_wheel">
         <visual>
             <geometry>
-                <cylinder radius = "0.05" length = "0.04"/>
+                <cylinder length="0.04" radius="0.05" />
             </geometry>
-            <material name = "blue"/>
+            <material name="blue"/>
         </visual>
         <collision>
             <geometry>
-                <cylinder radius = "0.05" length = "0.04"/>
+                <sphere radius="0.05" />
             </geometry>
         </collision>
-        <xacro:inertial_cylinder mass = "1.0" length = "0.04" radius = "0.05">
-            <origin xyz = "0 0 0" rpy = "0 0 0"/>
+        <xacro:inertial_cylinder mass="0.1" length="0.04" radius="0.05">
+            <origin xyz="0 0 0" rpy="0 0 0"/>
         </xacro:inertial_cylinder>
     </link>
-    <!-- CASTER WHEEL LINK-->
-    <joint name = "caster_wheel_joint" type = "fixed">
-        <parent link = "chassis"/>
-        <child link = "caster_wheel"/>
-        <origin xyz = "0.24 0 0"/>
+    <!-- CASTER WHEEL -->
+    <joint name="caster_wheel_joint" type="fixed">
+        <parent link="chassis"/>
+        <child link="caster_wheel"/>
+        <origin xyz="0.24 0 0" rpy="0 0 0"/>
     </joint>
-    <link name = "caster_wheel">
+    <link name="caster_wheel">
         <visual>
             <geometry>
-                <sphere radius = "0.05"/>
+                <sphere radius="0.05" />
             </geometry>
-            <material name = "black"/>
+            <material name="black"/>
         </visual>
         <collision>
             <geometry>
-                <sphere radius = "0.05"/>
+                <sphere radius="0.05" />
             </geometry>
         </collision>
-        <xacro:inertial_sphere mass = "1.0" radius = "0.05">
-            <origin xyz = "0 0 0" rpy = "0 0 0"/>
+        <xacro:inertial_sphere mass="0.1" radius="0.05">
+            <origin xyz="0 0 0" rpy="0 0 0"/>
         </xacro:inertial_sphere>
     </link>
+    <gazebo reference="caster_wheel">
+        <mu1 value="0.0"/>
+        <mu2 value="0.0"/>
+    </gazebo>
 </robot>
